File: design.kicad_sch (KiCad schematic)
At the start: 0 parts

Commit message: Update design.kicad_sch
Parts:
- added C?: 2.2uF, symbol Device:C_Small
- added C? (x2): 100pF, symbol Device:C_Small
- added C?: 4.7uF, symbol Device:C_Small
- added C?: 2.2pF, symbol Device:C_Small
- added D?: BAT54C, Package_TO_SOT_SMD:SOT-23, symbol Diode:BAT54C
- added J?: Conn_01x06_Male, symbol Connector:Conn_01x06_Male
- added JP?: Jumper_2_Open, symbol Jumper:Jumper_2_Open
- added R?: 47ohm, symbol Device:R_Small
- added R?: 470ohm, symbol Device:R_Small
- added R? (x2): 4.7k, symbol Device:R_Small
- added U?: IQS231A-00000000-TSR, IQS231A-00000000-TSR:SOT95P280X100-6N, symbol Sensor_Touch_custom:IQS231A-00000000-TSR
Connections:
- new net: C?.1, C?.1, R?.1, U?.5 (VDDHI)
- new net: C?.1, C?.1, U?.4 (VREG)
- new net: C?.1, R?.2, U?.6 (CX)
- new net: D?.1, J?.6 (Pin_6)
- new net CX: J?.5 (Pin_5), R?.1
- new net GND: C?.2, C?.2, C?.2, C?.2, C?.2, J?.4 (Pin_4), JP?.2 (B), U?.2 (VSS)
- new net IO1/SCL: D?.3, J?.2 (Pin_2), R?.1, U?.1 (IO1/SCL)
- new net IO2/SDA: J?.1 (Pin_1), JP?.1 (A), R?.1, U?.3 (IO2/SDA)
- new net VCC: J?.3 (Pin_3), R?.2, R?.2, R?.2
